File: fab/kicad/CON_1xIO_V2/CON_1xIO_V2.kicad_sch (KiCad schematic)
At the start: 8 parts, among them J1 Box_02x03_P2.54_Vertical, J3 Screw_Terminal_01x02_P5, J5 Screw_Terminal_01x02_P5, J6 Screw_Terminal_01x02_P5

Commit message: Update kicad-Files
Other:
- note added: "V2"
- moved on the sheet: J3
Changed lines of the file:
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@@
+	(wire
+		(pts
+			(xy 224.79 114.3) (xy 224.79 130.81)
+		)
+		(stroke
+			(width 0)
+			(type default)
+		)
+	)
 	(wire
 		(pts
@@
 	(wire
 		(pts
-			(xy 219.71 147.32) (xy 213.36 147.32)
+			(xy 219.71 144.78) (xy 213.36 144.78)
 		)
 		(stroke
@@
 	(wire
 		(pts
-			(xy 224.79 113.03) (xy 224.79 130.81)
-		)
-		(stroke
-			(width 0)
-			(type default)
-		)
-	)
-	(wire
-		(pts
-			(xy 222.25 113.03) (xy 222.25 119.38)
-		)
-		(stroke
-			(width 0)
-			(type default)
-		)
-	)
-	(wire
-		(pts
-			(xy 224.79 143.51) (xy 224.79 146.05)
-		)
-		(stroke
-			(width 0)
-			(type default)
-		)
-	)
-	(wire
-		(pts
-			(xy 228.6 119.38) (xy 228.6 146.05)
+			(xy 222.25 114.3) (xy 222.25 120.65)
+		)
+		(stroke
+			(width 0)
+			(type default)
+		)
+	)
+	(wire
+		(pts
+			(xy 224.79 143.51) (xy 224.79 144.78)
+		)
+		(stroke
+			(width 0)
+			(type default)
+		)
+	)
+	(wire
+		(pts
+			(xy 228.6 120.65) (xy 228.6 144.78)
 		)
 		(stroke
@@
 	(wire
 		(pts
-			(xy 219.71 143.51) (xy 219.71 147.32)
+			(xy 219.71 143.51) (xy 219.71 144.78)
 		)
 		(stroke
@@
 	(wire
 		(pts
-			(xy 228.6 146.05) (xy 224.79 146.05)
-		)
-		(stroke
-			(width 0)
-			(type default)
-		)
-	)
-	(wire
-		(pts
-			(xy 213.36 147.32) (xy 213.36 124.46)
-		)
-		(stroke
-			(width 0)
-			(type default)
-		)
-	)
-	(wire
-		(pts
-			(xy 222.25 119.38) (xy 228.6 119.38)
-		)
-		(stroke
-			(width 0)
-			(type default)
+			(xy 228.6 144.78) (xy 224.79 144.78)
+		)
+		(stroke
+			(width 0)
+			(type default)
+		)
+	)
+	(wire
+		(pts
+			(xy 213.36 144.78) (xy 213.36 124.46)
+		)
+		(stroke
+			(width 0)
+			(type default)
+		)
+	)
+	(wire
+		(pts
+			(xy 222.25 120.65) (xy 228.6 120.65)
+		)
+		(stroke
+			(width 0)
+			(type default)
+		)
+	)
+	(text "V2"
+		(exclude_from_sim no)
+		(at 207.01 137.922 0)
+		(effects
+			(font
+				(size 2.032 2.032)
+				(thickness 0.4064)
+				(bold yes)
+			)
 		)
 	)
@@
 	)
 	(label "C1+"
-		(at 222.25 118.11 90)
+		(at 222.25 119.38 90)
 		(effects
 			(font
@@
 	)
 	(label "C1-"
-		(at 224.79 118.11 90)
+		(at 224.79 119.38 90)
 		(effects
 			(font
@@
 	(symbol
 		(lib_id "_kh_library:Screw_Terminal_01x02_P5")
-		(at 222.25 107.95 90)
+		(at 222.25 109.22 90)
 		(unit 1)
 		(exclude_from_sim no)
@@
 		(dnp no)
 		(property "Reference" "J3"
-			(at 218.948 108.204 90)
+			(at 218.948 109.474 90)
 			(effects
 				(font
@@
 		)
 		(property "Value" "Screw_Terminal_01x02_P5"
-			(at 212.852 104.648 90)
+			(at 222.758 104.394 90)
 			(effects
 				(font
@@
 		)
 		(property "Footprint" "_kh_library:Screw_Terminal_01x02_P5"
-			(at 222.758 97.028 90)
+			(at 222.758 98.298 90)
 			(effects
 				(font
@@
 		)
 		(property "Datasheet" "~"
-			(at 222.25 107.95 0)
+			(at 222.25 109.22 0)
 			(effects
 				(font
@@
 		)
 		(property "Description" "Generic screw terminal, single row, 01x02"
-			(at 223.52 99.314 90)
+			(at 223.52 100.584 90)
 			(effects
 				(font
@@
 		)
 		(property "Value" "Box_02x03_P2.54_Vertical"
-			(at 216.154 151.13 90)
+			(at 221.488 149.352 90)
 			(effects
 				(font
@@
 		)
 		(property "Value" "Screw_Terminal_01x02_P5"
-			(at 245.11 125.476 90)
-			(effects
-				(font
+			(at 246.126 125.476 90)
+			(effects
+				(font
