File: fab/kicad/CON_6pol_6_V2/CON_6pol_6_V2.kicad_sch (KiCad schematic)
At the start: 7 parts, among them J5 Box_02x03_P2.54_Vertical, J6 Screw_Terminal_01x03_P5, J7 Screw_Terminal_01x03_P5

Commit message: Update kicad-Files
Other:
- note added: "V2"
Changed lines of the file:
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@@
+		)
+	)
+	(text "V2"
+		(exclude_from_sim no)
+		(at 212.344 131.826 0)
+		(effects
+			(font
+				(size 2.032 2.032)
+				(thickness 0.4064)
+				(bold yes)
+			)
 		)
 	)
