File: fab/kicad/3D/Stecker_SubD25_Klemme10_V1.kicad_sch (KiCad schematic)
At the start: 3 parts, among them J1 DB25_Plug, J2 Screw_Terminal_01x10, J3 Screw_Terminal_01x05

Commit message: Replace äöü
Other:
- note added: "N&ouml;rdliche Schiene, n&ouml;rdliches Gleis"
- note removed: "Nördliche Schiene, nördliches Gleis"
Changed lines of the file:
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@@
 		)
 	)
-	(text "Nördliche Schiene, nördliches Gleis"
+	(text "N&ouml;rdliche Schiene, n&ouml;rdliches Gleis"
 		(exclude_from_sim no)
 		(at 131.826 52.578 0)
