File: fab/kicad/CON_SubD_Screw10_V1/CON_SubD_Screw10_V1.kicad_sch (KiCad schematic)
At the start: 8 parts, among them J1 DB25_Plug, J2 Screw_Terminal_01x10_P5, J3 Conn_01x01_kh, J4 Conn_01x01_kh

Commit message: Replace äöü
Other:
- note added: "N&ouml;rdliche Schiene, n&ouml;rdliches Gleis"
- note added: "S&uuml;dliche Schiene, n&ouml;rdliches Gleis"
- note added: "S&uuml;dliche Schiene, s&uuml;dliches Gleis"
- note removed: "Nördliche Schiene, nördliches Gleis"
- note removed: "Südliche Schiene, nördliches Gleis"
- note removed: "Südliche Schiene, südliches Gleis"
Changed lines of the file:
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@@
 		)
 	)
-	(text "Südliche Schiene, südliches Gleis"
+	(text "S&uuml;dliche Schiene, s&uuml;dliches Gleis"
 		(exclude_from_sim no)
 		(at 113.03 81.788 0)
@@
 		)
 	)
-	(text "Südliche Schiene, nördliches Gleis"
+	(text "S&uuml;dliche Schiene, n&ouml;rdliches Gleis"
 		(exclude_from_sim no)
 		(at 113.03 61.468 0)
@@
 		)
 	)
-	(text "Nördliche Schiene, nördliches Gleis"
+	(text "N&ouml;rdliche Schiene, n&ouml;rdliches Gleis"
 		(exclude_from_sim no)
 		(at 113.03 58.928 0)
@@
 		)
 	)
-	(text "Südliche Schiene, nördliches Gleis"
+	(text "S&uuml;dliche Schiene, n&ouml;rdliches Gleis"
 		(exclude_from_sim no)
 		(at 113.03 79.248 0)
