File: fab/kicad/RW_5V_1OUT_LED_V2/RW_5V_1OUT_LED_V2.kicad_sch (KiCad schematic)
At the start: 18 parts, among them J1 Conn_01x08_Pin, J2 Conn_01x08_Pin, Q1 BC337

Commit message: Replace äöü
Parts:
- D3: value LED grün -> LED gr&uuml;n
Other:
- note added: "D2 zeigt, ob der Taster gedr&uuml;ckt ist. Kein Tastendruck ergibt REMOTE-Steuerung."
- note removed: "D2 zeigt, ob der Taster gedrückt ist. Kein Tastendruck ergibt REMOTE-Steuerung."
Changed lines of the file:
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@@
 		)
 	)
-	(text "D2 zeigt, ob der Taster gedrückt ist.\nKein Tastendruck ergibt REMOTE-Steuerung."
+	(text "D2 zeigt, ob der Taster gedr&uuml;ckt ist.\nKein Tastendruck ergibt REMOTE-Steuerung."
 		(exclude_from_sim no)
 		(at 112.268 139.7 0)
@@
 			)
 		)
-		(property "Value" "LED grün"
+		(property "Value" "LED gr&uuml;n"
 			(at 47.498 85.09 90)
 			(effects
