File: fab/kicad/RW_5V_2IO_LED_V2/RW_5V_2IO_LED_V2.kicad_pcb (KiCad board)
At the start: 2 copper layers, 41 x 41 mm, 22 parts, among them J1 Conn_01x08_Pin, J2 Conn_01x08_Pin, Q1 BC337, SW1 SW_Push_DPDT_8x8, SW2 SW_Push_DPDT_8x8

Commit message: Replace äöü
Parts:
- D3: value LED grün -> LED gr&uuml;n
Other:
- board text added: "LED gr&uuml;n"
- board text removed: "LED grün"
Changed lines of the file:
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@@
 			)
 		)
-		(property "Value" "LED grün"
+		(property "Value" "LED gr&uuml;n"
 			(at 1.27 3.302 0)
 			(layer "B.Fab")
@@
 		)
 	)
-	(gr_text "LED grün"
+	(gr_text "LED gr&uuml;n"
 		(at 38.1 52.705 0)
 		(layer "B.SilkS")
@@
 		)
 	)
-	(gr_text "LED grün"
+	(gr_text "LED gr&uuml;n"
 		(at 38.3794 52.7812 0)
 		(layer "F.SilkS")
