File: fab/kicad/RW_5V_2IO_LED_V2/RW_5V_2IO_LED_V2.kicad_sch (KiCad schematic)
At the start: 22 parts, among them J1 Conn_01x08_Pin, J2 Conn_01x08_Pin, Q1 BC337, SW1 SW_Push_DPDT_8x8, SW2 SW_Push_DPDT_8x8

Commit message: Replace äöü
Parts:
- D3: value LED grün -> LED gr&uuml;n
Changed lines of the file:
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@@
 			)
 		)
-		(property "Value" "LED grün"
+		(property "Value" "LED gr&uuml;n"
 			(at 47.498 85.09 90)
 			(effects
