File: fab/kicad/RW_5V_DPDT_LED_V1/RW_5V_DPDT_LED_V1.kicad_pcb (KiCad board)
At the start: 2 copper layers, 41 x 41 mm, 17 parts, among them J1 Conn_01x08_Pin, J2 Conn_01x08_Pin, SW2 SW_Push_DPDT_8x8, SW3 SW_Push_DPDT_8x8

Commit message: Replace äöü
Parts:
- D1, D3: value LED grün -> LED gr&uuml;n
Other:
- board text added: "LED gr&uuml;n"
- board text removed: "LED grün"
Changed lines of the file:
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@@
 			)
 		)
-		(property "Value" "LED grün"
+		(property "Value" "LED gr&uuml;n"
 			(at 1.524 3.302 0)
 			(layer "B.Fab")
@@
 			)
 		)
-		(property "Value" "LED grün"
+		(property "Value" "LED gr&uuml;n"
 			(at 1.27 3.302 0)
 			(layer "B.Fab")
@@
 		)
 	)
-	(gr_text "LED grün"
+	(gr_text "LED gr&uuml;n"
 		(at 38.1 52.578 0)
 		(layer "B.SilkS")
@@
 		)
 	)
-	(gr_text "LED grün"
+	(gr_text "LED gr&uuml;n"
 		(at 37.846 29.718 0)
 		(layer "B.SilkS")
