File: fab/kicad/RW_5V_DPDT_LED_V1/RW_5V_DPDT_LED_V1.kicad_sch (KiCad schematic)
At the start: 17 parts, among them J1 Conn_01x08_Pin, J2 Conn_01x08_Pin, SW2 SW_Push_DPDT_8x8, SW3 SW_Push_DPDT_8x8

Commit message: Update kicad files
Changed lines of the file:
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@@
 	(text "Manual"
 		(exclude_from_sim no)
-		(at 119.126 75.438 0)
+		(at 119.634 77.216 0)
 		(effects
 			(font
@@
 	(text "Remote-Local"
 		(exclude_from_sim no)
-		(at 153.67 75.438 0)
+		(at 154.178 77.216 0)
 		(effects
 			(font
@@
 	(text "Show Output"
 		(exclude_from_sim no)
-		(at 78.486 75.438 0)
+		(at 78.994 77.216 0)
 		(effects
 			(font

Commit message: Replace äöü
Parts:
- D1, D3: value LED grün -> LED gr&uuml;n
Changed lines of the file:
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@@
 			)
 		)
-		(property "Value" "LED grün"
+		(property "Value" "LED gr&uuml;n"
 			(at 95.758 88.9 90)
 			(effects
@@
 			)
 		)
-		(property "Value" "LED grün"
+		(property "Value" "LED gr&uuml;n"
 			(at 69.088 88.9 90)
 			(effects
