File: fab/kicad/RW_5V_W2_LED_V2/RW_5V_W2_LED_V2.kicad_pcb (KiCad board)
At the start: 2 copper layers, 41 x 41 mm, 31 parts, among them J1 Conn_01x08_Pin, J2 Conn_01x08_Pin, Q1 BC337, Q2 BC337, Q3 BC337, Q4 BC337

Commit message: Replace äöü
Parts:
- D2, D5: value LED grün -> LED gr&uuml;n
Other:
- board text added: "LED gr&uuml;n"
- board text removed: "LED grün"
Changed lines of the file:
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@@
 			)
 		)
-		(property "Value" "LED grün"
+		(property "Value" "LED gr&uuml;n"
 			(at 1.27 -2.96 0)
 			(layer "B.Fab")
@@
 			)
 		)
-		(property "Value" "LED grün"
+		(property "Value" "LED gr&uuml;n"
 			(at 1.27 -2.96 0)
 			(layer "B.Fab")
@@
 		)
 	)
-	(gr_text "LED grün"
+	(gr_text "LED gr&uuml;n"
 		(at 40.767 48.2346 0)
 		(layer "B.SilkS")
@@
 		)
 	)
-	(gr_text "LED grün"
+	(gr_text "LED gr&uuml;n"
 		(at 68.8848 48.2092 0)
 		(layer "B.SilkS")
@@
 		)
 	)
-	(gr_text "LED grün"
+	(gr_text "LED gr&uuml;n"
 		(at 67.3354 47.625 0)
 		(layer "F.SilkS")
@@
 		)
 	)
-	(gr_text "LED grün"
+	(gr_text "LED gr&uuml;n"
 		(at 37.8714 47.7774 0)
 		(layer "F.SilkS")
