File: fab/kicad/RW_5V_W2_LED_V2/RW_5V_W2_LED_V2.kicad_sch (KiCad schematic)
At the start: 31 parts, among them J1 Conn_01x08_Pin, J2 Conn_01x08_Pin, Q1 BC337, Q2 BC337, Q3 BC337, Q4 BC337

Commit message: Replace äöü
Parts:
- D2, D5: value LED grün -> LED gr&uuml;n
Other:
- note added: "Taster dr&uuml;cken bewirkt"
- note removed: "Taster drücken bewirkt"
Changed lines of the file:
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@@
 		)
 	)
-	(text "Taster drücken bewirkt"
+	(text "Taster dr&uuml;cken bewirkt"
 		(exclude_from_sim no)
 		(at 141.732 104.394 0)
@@
 			)
 		)
-		(property "Value" "LED grün"
+		(property "Value" "LED gr&uuml;n"
 			(at 156.972 55.88 0)
 			(effects
@@
 			)
 		)
-		(property "Value" "LED grün"
+		(property "Value" "LED gr&uuml;n"
 			(at 148.082 57.15 0)
 			(effects
