File: fab/kicad/RW_5V_W2_STRG_V2/RW_5V_W2_STRG_V2.kicad_sch (KiCad schematic)
At the start: 29 parts, among them J1 Conn_01x08_Pin, J2 Conn_01x08_Pin, J3 Box_02x03_P2.54_Vertical, J4 Box_02x05_P2.54_Vertical, J5 Box_02x03_P2.54_Vertical, K1 IM03TS, K3 IM03TS, Q1 BC327, Q2 BC327

Commit message: Replace äöü
Other:
- note added: "Zur LED-Anzeige/R&uuml;ckmeldung"
- note removed: "Zur LED-Anzeige/Rückmeldung"
Changed lines of the file:
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@@
 		)
 	)
-	(text "Zur LED-Anzeige/Rückmeldung"
+	(text "Zur LED-Anzeige/R&uuml;ckmeldung"
 		(exclude_from_sim no)
 		(at 113.792 158.75 0)
