File: fab/kicad/RW_5V_W3_LED_V4/RW_5V_W3_LED_V4.kicad_sch (KiCad schematic)
At the start: 41 parts, among them J1 Conn_01x08_Pin, J2 Conn_01x08_Pin, J3 Jumper_2, J4 Jumper_2, Q1 BC337, Q2 BC337, Q3 BC337, Q4 BC337, Q5 BC337, Q6 BC337

Commit message: Replace äöü
Parts:
- D2, D5: value LED grün -> LED gr&uuml;n
Changed lines of the file:
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@@
 			)
 		)
-		(property "Value" "LED grün"
+		(property "Value" "LED gr&uuml;n"
 			(at 148.59 52.3874 90)
 			(effects
@@
 			)
 		)
-		(property "Value" "LED grün"
+		(property "Value" "LED gr&uuml;n"
 			(at 142.24 52.3874 90)
 			(effects
