File: fab/kicad/RW_5V_W3_LED_V5/RW_5V_W3_LED_V5.kicad_pcb (KiCad board)
At the start: 2 copper layers, 41 x 41 mm, 41 parts, among them J1 Conn_01x08_Pin, J2 Conn_01x08_Pin, J3 Jumper_2, J4 Jumper_2, Q1 BC337, Q2 BC337, Q3 BC337, Q4 BC337, Q5 BC337, Q6 BC337

Commit message: Replace äöü
Parts:
- D2, D5: value LED grün -> LED gr&uuml;n
Other:
- board text added: "LED gr&uuml;n"
- board text removed: "LED grün"
Changed lines of the file:
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@@
 			)
 		)
-		(property "Value" "LED grün"
+		(property "Value" "LED gr&uuml;n"
 			(at 1.27 -2.96 0)
 			(layer "B.Fab")
@@
 			)
 		)
-		(property "Value" "LED grün"
+		(property "Value" "LED gr&uuml;n"
 			(at 1.27 -2.96 180)
 			(layer "B.Fab")
@@
 		)
 	)
-	(gr_text "LED grün"
+	(gr_text "LED gr&uuml;n"
 		(at 35.56 47.625 0)
 		(layer "B.SilkS")
@@
 		)
 	)
-	(gr_text "LED grün"
+	(gr_text "LED gr&uuml;n"
 		(at 61.214 46.736 0)
 		(layer "B.SilkS")
