File: fab/kicad/RW_5V_W3_STRG_V4/RW_5V_W3_STRG_V4.kicad_sch (KiCad schematic)
At the start: 41 parts, among them J1 Conn_01x08_Pin, J2 Conn_01x08_Pin, J3 Box_02x03_P2.54_Vertical, J4 Box_02x05_P2.54_Vertical, J5 Box_02x03_P2.54_Vertical, K1 IM03TS, K2 IM03TS, K3 IM03TS, K4 IM03TS, Q1 BC327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

Commit message: Replace äöü
Other:
- note added: "LED-Anzeige/R&uuml;ckmeldung"
- note removed: "LED-Anzeige/Rückmeldung"
Changed lines of the file:
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@@
 		)
 	)
-	(text "LED-Anzeige/Rückmeldung"
+	(text "LED-Anzeige/R&uuml;ckmeldung"
 		(exclude_from_sim no)
 		(at 120.142 158.75 0)
