File: fab/kicad/RW_5V_SUB25_10_east_V4/RW_5V_SUB25_10_east_V4.kicad_sch (KiCad schematic)
At the start: 13 parts, among them J1 DB25_Plug, J10 Screw_Terminal_01x02_P5, J2 Screw_Terminal_01x10_P5, J5 Conn_01x06, J6 Conn_01x06, J7 Screw_Terminal_01x02_P5, J8 Screw_Terminal_01x02_P5, J9 Screw_Terminal_01x02_P5

Commit message: Update LIESMICH.md
Other:
- note added: "N&ouml;rdliche Schiene, n&ouml;rdliches Gleis"
- note added: "S&uuml;dliche Schiene, n&ouml;rdliches Gleis"
- note added: "S&uuml;dliche Schiene, s&uuml;dliches Gleis"
- note removed: "Nördliche Schiene, nördliches Gleis"
- note removed: "Südliche Schiene, nördliches Gleis"
- note removed: "Südliche Schiene, südliches Gleis"
Changed lines of the file:
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@@
 		)
 	)
-	(text "Südliche Schiene, südliches Gleis"
+	(text "S&uuml;dliche Schiene, s&uuml;dliches Gleis"
 		(exclude_from_sim no)
 		(at 113.03 84.328 0)
@@
 		)
 	)
-	(text "Südliche Schiene, nördliches Gleis"
+	(text "S&uuml;dliche Schiene, n&ouml;rdliches Gleis"
 		(exclude_from_sim no)
 		(at 113.03 61.468 0)
@@
 		)
 	)
-	(text "Nördliche Schiene, nördliches Gleis"
+	(text "N&ouml;rdliche Schiene, n&ouml;rdliches Gleis"
 		(exclude_from_sim no)
 		(at 113.284 55.88 0)
@@
 		)
 	)
-	(text "Südliche Schiene, nördliches Gleis"
+	(text "S&uuml;dliche Schiene, n&ouml;rdliches Gleis"
 		(exclude_from_sim no)
 		(at 113.03 79.248 0)
