File: fab/kicad/dcc_track_UI_detection_V2/dcc_track_UI_detection_V2.kicad_pcb (KiCad board)
At the start: 2 copper layers, 99.1 x 33 mm, 49 parts, among them J1 Screw_Terminal_01x02_P5, J2 Screw_Terminal_01x02_P5, J3 Jumper_2, J5 Box_02x03_P2.54_Vertical, Q1 BC337, Q2 BC337, U1 INA333_Board, U2 LM393, U3 SFH615A

Commit message: Update rcc6.../LIESMICH.md
Parts:
- R5: value 33k -> 47k
- R8: value 4k7 -> 1k
Other:
- board text added: "+"
- board text added: "260710 KH"
- board text added: "260710KH"
- board text removed: "260709 KH"
- board text removed: "260709KH"
Changed lines of the file:
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@@
 			)
 		)
-		(property "Value" "4k7"
+		(property "Value" "1k"
 			(at -3.683 0 0)
 			(layer "F.SilkS")
@@
 			)
 		)
-		(property "Value" "33k"
+		(property "Value" "47k"
 			(at 3.683 0 90)
 			(layer "F.SilkS")
@@
 		(tags "Resistor Axial_DIN0204 series Axial Vertical pin pitch 2.54mm 0.167W length 3.6mm diameter 1.6mm")
 		(property "Reference" "C5"
-			(at 0.254 -3.048 0)
+			(at 0.508 -2.794 0)
 			(layer "F.SilkS")
 			(effects
@@
 		)
 		(property "Value" "10u"
-			(at 1.778 -3.048 0)
+			(at 2.032 -3.048 0)
 			(layer "F.SilkS")
 			(effects
@@
 		)
 		(fp_text user "${REFERENCE}"
-			(at 0.254 -3.048 0)
+			(at 0.508 -2.794 0)
 			(layer "F.Fab")
 			(effects
@@
 		)
 	)
-	(gr_text "260709KH"
+	(gr_text "260710KH"
 		(at 59.944 82.169 0)
 		(layer "F.Cu")
@@
 		)
 	)
-	(gr_text "260709 KH"
+	(gr_text "260710 KH"
 		(at 60.198 82.169 0)
 		(layer "B.Cu")
@@
 		)
 	)
-	(gr_text "260709KH"
+	(gr_text "260710KH"
 		(at 108.204 81.534 0)
 		(layer "F.SilkS")
@@
 	)
 	(gr_text "DCC1_OUT"
-		(at 144.018 60.706 0)
+		(at 144.018 60.198 0)
 		(layer "F.SilkS")
 		(effects
@@
 		)
 	)
+	(gr_text "+"
+		(at 97.536 72.136 0)
+		(layer "F.SilkS")
+		(effects
+			(font
+				(size 1.5 1.5)
+				(thickness 0.3)
+				(bold yes)
+			)
+			(justify left bottom)
+		)
+	)
+	(gr_text "+"
+		(at 137.668 63.246 0)
+		(layer "F.SilkS")
+		(effects
+			(font
+				(size 1.5 1.5)
+				(thickness 0.3)
+				(bold yes)
+			)
+			(justify left bottom)
+		)
+	)
 	(gr_text "DCC1_IN"
 		(at 55.88 60.198 0)
@@
 		)
 	)
-	(gr_text "260709KH"
+	(gr_text "260710KH"
 		(at 108.204 81.534 0)
 		(layer "B.SilkS")
