File: fab/kicad/dcc_track_UI_detection_V2/dcc_track_UI_detection_V2.kicad_sch (KiCad schematic)
At the start: 49 parts, among them J1 Screw_Terminal_01x02_P5, J2 Screw_Terminal_01x02_P5, J3 Jumper_2, J5 Box_02x03_P2.54_Vertical, Q1 BC337, Q2 BC337, U1 INA333_Board, U2 LM393, U3 SFH615A

Commit message: Update rcc6.../LIESMICH.md
Parts:
- R5: value 33k -> 47k
- R8: value 4k7 -> 1k
Other:
- note added: "dcc_track_UI_detection_V2 2026-07-10"
- note removed: "dcc_track_UI_detection_V1 2026-07-09"
- moved on the sheet: C6, C7, C8, D1, D2, D4, D5, D6, J1, J2, J3, J5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
