File: fab/kicad/RCC_RGY_TVn_LED_V2/RCC_RGY_TVn_LED_V2.kicad_pcb (KiCad board)
At the start: 2 copper layers, 41 x 41 mm, 34 parts, among them J1 Conn_01x08_Pin, J2 Conn_01x08_Pin, Q1 BC337, Q2 BC327, Q3 BC327, Q4 BC327, Q5 BC327, Q6 BC337, SW1 SW_Push_DPDT_8x8, SW2 SW_Push_DPDT_8x8

Commit message: Update RCC_GRY_*
Parts:
- R9: value 10k -> 47
- renumbered SW2 to SW3
Other:
- board text added: "RCC_RGY_TVn_LED_V2 260823KH"
- board text added: "SW3"
- board text removed: "260820 KH"
- board text removed: "RCC_RGY_TVn_LED_V1"
- board text removed: "SW2"
