File: fab/kicad/RCC_RGY_TVn_LED_V2/RCC_RGY_TVn_LED_V2.kicad_sch (KiCad schematic)
At the start: 34 parts, among them J1 Conn_01x08_Pin, J2 Conn_01x08_Pin, Q1 BC337, Q2 BC327, Q3 BC327, Q4 BC327, Q5 BC327, Q6 BC337, SW1 SW_Push_DPDT_8x8, SW2 SW_Push_DPDT_8x8

Commit message: Update RCC_GRY_*
Parts:
- R9: value 10k -> 47
- renumbered SW2 to SW3
Other:
- note added: "RCC_RGY_TVn_LED_V2 2026-08-23"
- note removed: "RCC_RGY_TVn_LED_V1 2026-08-20"
Changed lines of the file:
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@@
 		)
 	)
-	(text "RCC_RGY_TVn_LED_V1\n2026-08-20"
+	(text "RCC_RGY_TVn_LED_V2\n2026-08-23"
 		(exclude_from_sim no)
 		(at 229.362 132.08 0)
@@
 		)
 		(instances
-			(project "RCC_RGY_TVn_LED_V1"
+			(project "RCC_RGY_TVn_LED_V2"
 				(path "/4d39acef-efca-4909-8928-de8e022e1cdc"
 					(reference "D4")
@@
 		)
 		(instances
-			(project "RCC_RGY_TVn_LED_V1"
+			(project "RCC_RGY_TVn_LED_V2"
 				(path "/4d39acef-efca-4909-8928-de8e022e1cdc"
 					(reference "R8")
@@
 		)
 		(instances
-			(project "RCC_RGY_TVn_LED_V1"
+			(project "RCC_RGY_TVn_LED_V2"
 				(path "/4d39acef-efca-4909-8928-de8e022e1cdc"
 					(reference "D2")
@@
 		)
 		(instances
-			(project "RCC_RGY_TVn_LED_V1"
+			(project "RCC_RGY_TVn_LED_V2"
 				(path "/4d39acef-efca-4909-8928-de8e022e1cdc"
 					(reference "R12")
@@
 		)
 		(instances
-			(project "RCC_RGY_TVn_LED_V1"
+			(project "RCC_RGY_TVn_LED_V2"
 				(path "/4d39acef-efca-4909-8928-de8e022e1cdc"
 					(reference "R7")
@@
 		)
 		(instances
-			(project "RCC_RGY_TVn_LED_V1"
+			(project "RCC_RGY_TVn_LED_V2"
 				(path "/4d39acef-efca-4909-8928-de8e022e1cdc"
 					(reference "Q6")
@@
 		)
 		(instances
-			(project "RCC_RGY_TVn_LED_V1"
+			(project "RCC_RGY_TVn_LED_V2"
 				(path "/4d39acef-efca-4909-8928-de8e022e1cdc"
 					(reference "R2")
@@
 		)
 		(instances
-			(project "RCC_RGY_TVn_LED_V1"
+			(project "RCC_RGY_TVn_LED_V2"
 				(path "/4d39acef-efca-4909-8928-de8e022e1cdc"
 					(reference "D1")
@@
 		)
 		(instances
-			(project "RCC_RGY_TVn_LED_V1"
+			(project "RCC_RGY_TVn_LED_V2"
 				(path "/4d39acef-efca-4909-8928-de8e022e1cdc"
 					(reference "R5")
@@
 		)
 		(instances
-			(project "RCC_RGY_TVn_LED_V1"
+			(project "RCC_RGY_TVn_LED_V2"
 				(path "/4d39acef-efca-4909-8928-de8e022e1cdc"
 					(reference "R1")
@@
 		)
 		(instances
-			(project "RCC_RGY_TVn_LED_V1"
+			(project "RCC_RGY_TVn_LED_V2"
 				(path "/4d39acef-efca-4909-8928-de8e022e1cdc"
 					(reference "R14")
@@
 		)
 		(instances
-			(project "RCC_RGY_TVn_LED_V1"
+			(project "RCC_RGY_TVn_LED_V2"
 				(path "/4d39acef-efca-4909-8928-de8e022e1cdc"
 					(reference "R11")
@@
 		)
 		(instances
-			(project "RCC_RGY_TVn_LED_V1"
+			(project "RCC_RGY_TVn_LED_V2"
 				(path "/4d39acef-efca-4909-8928-de8e022e1cdc"
 					(reference "D3")
@@
 		)
 		(instances
-			(project "RCC_RGY_TVn_LED_V1"
+			(project "RCC_RGY_TVn_LED_V2"
 				(path "/4d39acef-efca-4909-8928-de8e022e1cdc"
 					(reference "H1")
@@
 		(in_pos_files yes)
 		(dnp no)
-		(property "Reference" "SW2"
+		(property "Reference" "SW3"
 			(at 247.396 75.946 0)
 			(show_name no)
@@
 		)
 		(instances
-			(project "RCC_RGY_TVn_LED_V1"
+			(project "RCC_RGY_TVn_LED_V2"
 				(path "/4d39acef-efca-4909-8928-de8e022e1cdc"
-					(reference "SW2")
+					(reference "SW3")
 					(unit 1)
 				)
@@
 		)
 		(instances
-			(project "RCC_RGY_TVn_LED_V1"
+			(project "RCC_RGY_TVn_LED_V2"
 				(path "/4d39acef-efca-4909-8928-de8e022e1cdc"
 					(reference "Q4")
@@
 		)
 		(instances
-			(project "RCC_RGY_TVn_LED_V1"
+			(project "RCC_RGY_TVn_LED_V2"
 				(path "/4d39acef-efca-4909-8928-de8e022e1cdc"
 					(reference "Q3")
@@
 		)
 		(instances
-			(project "RCC_RGY_TVn_LED_V1"
+			(project "RCC_RGY_TVn_LED_V2"
 				(path "/4d39acef-efca-4909-8928-de8e022e1cdc"
 					(reference "Q2")
@@
 		)
 		(instances
-			(project "RCC_RGY_TVn_LED_V1"
+			(project "RCC_RGY_TVn_LED_V2"
 				(path "/4d39acef-efca-4909-8928-de8e022e1cdc"
 					(reference "R15")
@@
 		)
 		(instances
-			(project "RCC_RGY_TVn_LED_V1"
+			(project "RCC_RGY_TVn_LED_V2"
 				(path "/4d39acef-efca-4909-8928-de8e022e1cdc"
 					(reference "H3")
@@
 		)
 		(instances
-			(project "RCC_RGY_TVn_LED_V1"
+			(project "RCC_RGY_TVn_LED_V2"
 				(path "/4d39acef-efca-4909-8928-de8e022e1cdc"
 					(reference "H2")
@@
 		)
 		(instances
-			(project "RCC_RGY_TVn_LED_V1"
+			(project "RCC_RGY_TVn_LED_V2"
 				(path "/4d39acef-efca-4909-8928-de8e022e1cdc"
 					(reference "H4")
@@
 		)
 		(instances
-			(project "RCC_RGY_TVn_LED_V1"
+			(project "RCC_RGY_TVn_LED_V2"
 				(path "/4d39acef-efca-4909-8928-de8e022e1cdc"
 					(reference "R13")
@@
 		)
 		(instances
-			(project "RCC_RGY_TVn_LED_V1"
+			(project "RCC_RGY_TVn_LED_V2"
 				(path "/4d39acef-efca-4909-8928-de8e022e1cdc"
 					(reference "J2")
@@
 		)
 		(instances
-			(project "RCC_RGY_TVn_LED_V1"
+			(project "RCC_RGY_TVn_LED_V2"
 				(path "/4d39acef-efca-4909-8928-de8e022e1cdc"
 					(reference "C1")
@@
 		)
 		(instances
-			(project "RCC_RGY_TVn_LED_V1"
+			(project "RCC_RGY_TVn_LED_V2"
 				(path "/4d39acef-efca-4909-8928-de8e022e1cdc"
 					(reference "R10")
@@
 		)
 		(instances
-			(project "RCC_RGY_TVn_LED_V1"
+			(project "RCC_RGY_TVn_LED_V2"
 				(path "/4d39acef-efca-4909-8928-de8e022e1cdc"
 					(reference "Q1")
@@
 		)
 		(instances
-			(project "RCC_RGY_TVn_LED_V1"
+			(project "RCC_RGY_TVn_LED_V2"
 				(path "/4d39acef-efca-4909-8928-de8e022e1cdc"
 					(reference "R6")
@@
 		)
 		(instances
-			(project "RCC_RGY_TVn_LED_V1"
+			(project "RCC_RGY_TVn_LED_V2"
 				(path "/4d39acef-efca-4909-8928-de8e022e1cdc"
 					(reference "R3")
@@
 		)
 		(instances
-			(project "RCC_RGY_TVn_LED_V1"
+			(project "RCC_RGY_TVn_LED_V2"
 				(path "/4d39acef-efca-4909-8928-de8e022e1cdc"
 					(reference "SW1")
@@
 		)
 		(instances
-			(project "RCC_RGY_TVn_LED_V1"
+			(project "RCC_RGY_TVn_LED_V2"
 				(path "/4d39acef-efca-4909-8928-de8e022e1cdc"
 					(reference "R4")
@@
 			)
 		)
-		(property "Value" "10k"
+		(property "Value" "47"
 			(at 163.83 66.04 90)
 			(show_name no)
@@
 		)
 		(instances
-			(project "RCC_RGY_TVn_LED_V1"
+			(project "RCC_RGY_TVn_LED_V2"
 				(path "/4d39acef-efca-4909-8928-de8e022e1cdc"
 					(reference "R9")
@@
 		)
 		(instances
-			(project "RCC_RGY_TVn_LED_V1"
+			(project "RCC_RGY_TVn_LED_V2"
 				(path "/4d39acef-efca-4909-8928-de8e022e1cdc"
 					(reference "Q5")
@@
 		)
 		(instances
-			(project "RCC_RGY_TVn_LED_V1"
+			(project "RCC_RGY_TVn_LED_V2"
 				(path "/4d39acef-efca-4909-8928-de8e022e1cdc"
 					(reference "J1")
