File: fab/kicad/RCC_TUI_M_LED_V1/RCC_TUI_M_LED_V1.kicad_pcb (KiCad board)
At the start: 2 copper layers, 41 x 41 mm, 39 parts, among them J1 Conn_01x08_Pin, J2 Conn_01x08_Pin, Q1 BC337, Q2 BC337, Q3 BC337, Q4 BC337, Q5 BC337, SW1 SW_Push_DPDT_8x8, SW2 SW_Push_DPDT_8x8

Commit message: Add kicad files
Parts:
- removed Q5: BC337, _kh_library:TO-92_Inline_Wide_custom
- removed the R12 at (45.0, 42.4)
- removed the R5 at (44.0, 31.0)
- removed the R7 at (51.7, 42.4)
- added R10: 100k, Resistor_THT:R_Axial_DIN0204_L3.6mm_D1.6mm_P2.54mm_Vertical, F.Cu at (48.9, 47.8)
- added R13: 100k, Resistor_THT:R_Axial_DIN0204_L3.6mm_D1.6mm_P2.54mm_Vertical, F.Cu at (53.2, 44.6)
- added R3: 100k, Resistor_THT:R_Axial_DIN0204_L3.6mm_D1.6mm_P2.54mm_Vertical, F.Cu at (42.3, 40.1)
- added R6: 100k, Resistor_THT:R_Axial_DIN0204_L3.6mm_D1.6mm_P2.54mm_Vertical, F.Cu at (55.4, 44.6)
- Q1, Q2, Q3, Q4: value BC337 -> BS170
- R1: value 100k -> 10k
- R2, R9: value 10k -> 1k
- R8: value 47k -> 10k
- moved C1 10.1 mm to (55.4, 50.4)
- moved R14 4.65 mm to (41.5, 53.1), turned to -90 degrees
- moved R7 3.53 mm to (64.6, 27.9), turned to -90 degrees
- moved Q2 2.71 mm to (60.2, 42.0)
- moved R15 1.83 mm to (41.5, 57.7)
- moved R9 1.40 mm to (39.4, 50.8)
- moved R8 1.27 mm to (34.8, 50.7)
- moved Q3 0.52 mm to (45.1, 45.1)
- moved R16 0.39 mm to (62.5, 31.6)
- moved Q4 0.38 mm to (45.3, 58.8)
- moved Q1 0.13 mm to (44.8, 33.0)
- renumbered R10 to R11, R11 to R12, R13 to R14, R14 to R15, R15 to R16, R16 to R17, R3 to R4, R4 to R5, R6 to R7
Connections:
- net /Q1B renamed Net-(Q1-G)
- net /Q3B renamed Net-(Q3-G)
- Q2 pad 1: Net-(Q2-C) -> /RTViin
- Q2 pad 2: Net-(Q2-B) -> /TVi
- Q3 pad 3: /TViin -> /RTViin
- Q4 pad 2: /Q4B -> /FREi
- Q4 pad 3: /TViin -> /RTViin
- R16 pad 1: Net-(Q2-C) -> /RTViin
- R7 pad 2: Net-(Q2-C) -> /RTViin
Routing:
- net /RTViin: track 0.00 -> 38.8 mm
- net /FREi: track 5.28 -> 27.4 mm
- net Net-(Q2-B): track 21.2 -> 0.00 mm
- net /Q4B: track 15.4 -> 0.00 mm
- net Net-(Q2-C): track 11.7 -> 0.00 mm
- net /V_I2C: track 106.4 -> 97.7 mm
- net /TViin: track 8.45 -> 0.00 mm
- net /TVi: track 19.5 -> 26.9 mm
- net /S1ii: track 29.2 -> 35.8 mm
- net Net-(Q3-G): track 3.61 -> 8.58 mm
- net /TVii: track 3.68 -> 0.00 mm
- net Net-(Q1-G): track 3.87 -> 6.24 mm
- net /TVin: track 35.5 -> 37.8 mm
- net /RFREiin: track 45.7 -> 47.2 mm
- net /IONin: track 51.8 -> 50.6 mm
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Other:
- board text added: "RCC_TUI_M_LED_V1 260905 KH"
- board text removed: "BC337"
- board text removed: "RCC_TUI_B_LED_V1 260905 KH"
