File: fab/kicad/RCC_TUI_M_LED_V1/RCC_TUI_M_LED_V1.kicad_sch (KiCad schematic)
At the start: 39 parts, among them J1 Conn_01x08_Pin, J2 Conn_01x08_Pin, Q1 BC337, Q2 BC337, Q3 BC337, Q4 BC337, Q5 BC337, SW1 SW_Push_DPDT_8x8, SW2 SW_Push_DPDT_8x8

Commit message: Add kicad files
Parts:
- removed Q1, Q2, Q3, Q4, Q5: BC337, _kh_library:TO-92_Inline_Wide_custom, symbol Transistor_BJT:BC337
- removed R12, R5: 47k, _kh_library:R_Axial_DIN0204_L3.6mm_D1.6mm_P2.54mm_Vertical_kh, symbol Device:R
- removed R7: 10k, _kh_library:R_Axial_DIN0204_L3.6mm_D1.6mm_P2.54mm_Vertical_kh, symbol Device:R
- added Q1, Q2, Q3, Q4: BS170, _kh_library:TO-92_Inline_Wide_custom, symbol _kh_library:BS170_kh
- added R10, R13, R3, R6: 100k, Resistor_THT:R_Axial_DIN0204_L3.6mm_D1.6mm_P2.54mm_Vertical, symbol Device:R
- R1: value 100k -> 10k
- R2, R9: value 10k -> 1k
- R8: value 47k -> 10k
- renumbered R10 to R11, R11 to R12, R13 to R14, R14 to R15, R15 to R16, R16 to R17, R3 to R4, R4 to R5, R6 to R7
Connections:
- net 0V: now also Q1.3 (S), Q2.3 (S), R10.2, R13.2, R3.2, R6.2
- net FREi: now also Q3.1 (D), Q4.2 (G), R13.1
- net RFREiin: now also Q4.1 (D)
- net TVi: now also Q1.1 (D), Q2.2 (G), R6.1
- net RTViin: now reaches R16.1, R7.2
- net RTViin: now also Q2.1 (D), Q3.3 (S), Q4.3 (S)
- net Q1B: no longer names the net of R2.2
- net Q1B: now also Q1.2 (G), R3.1
- net Q3B: no longer names the net of R9.2
- net Q3B: now also Q3.2 (G), R10.1
Other:
- note added: "RCC_TUI_M_LED_V1 2026-09-05"
- note removed: "RCC_TUI_B_LED_V1 2026-09-05"
- moved on the sheet: R1, R16, R2, R4, R7
