File: fab/kicad/CON_20_3x_2x6pol_R_V1/CON_20_3x_2x6pol_R_V1.kicad_pcb (KiCad board)
At the start: 2 copper layers, 109 x 35 mm, 19 parts, among them J1 Box_02x03_P2.54_Vertical, J10 Box_02x10_P2.54_RCC, J11 Box_02x10_P2.54_RCC, J2 Box_02x03_P2.54_Vertical_kh, J4 Box_02x10_P2.54_RCC, J5 Conn_01x06, J6 Conn_01x06, J7 Screw_Terminal_01x02_P5, J8 Screw_Terminal_01x02_P5, J9 Screw_Terminal_01x02_P5, U1 DCDC_StepDown_LM2596

Commit message: Add some kicad files
Parts:
- moved H1 0.50 mm to (27.9, 47.2)
- moved H2 0.50 mm to (121.0, 47.2)
- moved H3 0.50 mm to (27.9, 77.2)
- moved H4 0.50 mm to (121.0, 77.2)
Other:
- board size 109 x 35 mm -> 109 x 36 mm
- board text added: "CON_20_3x_2x6pol_R_V1 261021 KH"
- board text removed: "CON_20_3x_2x6pol_R_V1 261018 KH"
- board text removed: "CON_20_3x_2x6pol_R_V1 261019 KH"
Changed lines of the file:
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@@
 	(footprint "MountingHole:MountingHole_2.7mm_M2.5_DIN965_Pad_TopBottom"
 		(layer "F.Cu")
-		(at 120.95 47.73)
+		(at 120.95 47.23)
 		(descr "Mounting Hole 2.7mm, M2.5, generated by kicad-footprint-generator mountinghole.py")
 		(tags "mountinghole M2.5 DIN965")
 		(property "Reference" "H2"
-			(at 2.342 -2.264 0)
+			(at 2.748 -1.891 0)
 			(layer "F.SilkS")
 			(effects
@@
 	(footprint "MountingHole:MountingHole_2.7mm_M2.5_DIN965_Pad_TopBottom"
 		(layer "F.Cu")
-		(at 120.95 76.73)
+		(at 120.95 77.23)
 		(descr "Mounting Hole 2.7mm, M2.5, generated by kicad-footprint-generator mountinghole.py")
 		(tags "mountinghole M2.5 DIN965")
@@
 	(footprint "MountingHole:MountingHole_2.7mm_M2.5_DIN965_Pad_TopBottom"
 		(layer "F.Cu")
-		(at 27.95 76.73)
+		(at 27.95 77.23)
 		(descr "Mounting Hole 2.7mm, M2.5, generated by kicad-footprint-generator mountinghole.py")
 		(tags "mountinghole M2.5 DIN965")
@@
 		)
 		(property "Value" "1000uF/35V"
-			(at 18.923 -0.254 0)
+			(at 20.193 -0.127 0)
 			(layer "F.SilkS")
 			(effects
@@
 	(footprint "MountingHole:MountingHole_2.7mm_M2.5_DIN965_Pad_TopBottom"
 		(layer "F.Cu")
-		(at 27.95 47.73)
+		(at 27.95 47.23)
 		(descr "Mounting Hole 2.7mm, M2.5, generated by kicad-footprint-generator mountinghole.py")
 		(tags "mountinghole M2.5 DIN965")
@@
 	)
 	(gr_rect
-		(start 24.95 44.73)
-		(end 133.95 79.73)
+		(start 24.95 44.23)
+		(end 133.95 80.23)
 		(stroke
 			(width 0.05)
@@
 		(layer "Edge.Cuts")
 	)
-	(gr_text "CON_20_3x_2x6pol_R_V1 261019 KH"
-		(at 49.022 51.562 0)
+	(gr_text "CON_20_3x_2x6pol_R_V1 261021 KH"
+		(at 48.006 51.943 0)
 		(layer "F.Cu")
 		(effects
@@
 		)
 	)
-	(gr_text "CON_20_3x_2x6pol_R_V1 261019 KH"
-		(at 76.962 51.562 0)
+	(gr_text "CON_20_3x_2x6pol_R_V1 261021 KH"
+		(at 75.946 51.943 0)
 		(layer "B.Cu")
 		(effects
@@
 		)
 	)
-	(gr_text "CON_20_3x_2x6pol_R_V1 261018 KH"
-		(at 25.654 51.308 270)
+	(gr_text "CON_20_3x_2x6pol_R_V1 261021 KH"
+		(at 25.908 49.657 270)
 		(layer "F.SilkS")
 		(effects
 			(font
-				(size 1.5 0.8)
+				(size 2 0.9)
 				(thickness 0.16)
 				(bold yes)
@@
 		)
 	)
-	(gr_text "CON_20_3x_2x6pol_R_V1 261018 KH"
-		(at 25.654 73.66 270)
+	(gr_text "CON_20_3x_2x6pol_R_V1 261021 KH"
+		(at 25.908 74.803 270)
 		(layer "B.SilkS")
 		(effects
 			(font
-				(size 1.5 0.8)
+				(size 2 0.9)
 				(thickness 0.16)
 				(bold yes)
@@
 	)
 	(segment
+		(start 125.705 55.905)
+		(end 125.222 56.388)
+		(width 1.6)
+		(layer "F.Cu")
+		(net "/WA")
+	)
+	(segment
 		(start 116.078 55.88)
 		(end 116.586 56.388)
@@
 	)
 	(segment
-		(start 125.222 56.134)
-		(end 125.451 55.905)
+		(start 127.405 55.905)
+		(end 125.705 55.905)
 		(width 1.6)
 		(layer "F.Cu")
@@
 	)
 	(segment
-		(start 125.451 55.905)
-		(end 127.405 55.905)
-		(width 1.6)
-		(layer "F.Cu")
-		(net "/WA")
-	)
-	(segment
 		(start 75.692 60.96)
 		(end 73.66 62.992)
@@
 		(net "/WA")
 	)
-	(segment
-		(start 125.222 56.388)
-		(end 125.222 56.134)
-		(width 1.6)
-		(layer "F.Cu")
-		(net "/WA")
-	)
 	(via
 		(at 73.66 62.992)
@@
 	)
 	(segment
-		(start 125.476 55.88)
-		(end 125.501 55.905)
+		(start 116.078 55.88)
+		(end 116.586 56.388)
 		(width 1.6)
 		(layer "B.Cu")
@@
 	)
 	(segment
-		(start 104.634 55.88)
-		(end 111.389 55.88)
+		(start 125.705 55.905)
+		(end 125.222 56.388)
 		(width 1.6)
 		(layer "B.Cu")
@@
 	)
 	(segment
-		(start 116.586 56.388)
-		(end 124.968 56.388)
+		(start 104.634 55.88)
+		(end 111.389 55.88)
 		(width 1.6)
 		(layer "B.Cu")
@@
 	)
 	(segment
-		(start 114.3 55.88)
-		(end 116.078 55.88)
+		(start 35.56 75.184)
+		(end 36.322 75.946)
 		(width 1.6)
 		(layer "B.Cu")
@@
 	)
 	(segment
-		(start 35.56 75.184)
-		(end 36.322 75.946)
+		(start 114.3 55.88)
+		(end 116.078 55.88)
 		(width 1.6)
 		(layer "B.Cu")
@@
 	)
 	(segment
-		(start 116.078 55.88)
-		(end 116.586 56.388)
+		(start 116.586 56.388)
+		(end 125.222 56.388)
 		(width 1.6)
 		(layer "B.Cu")
@@
 	)
 	(segment
-		(start 85.09 55.88)
-		(end 75.692 55.88)
+		(start 127.405 55.905)
+		(end 125.705 55.905)
 		(width 1.6)
 		(layer "B.Cu")
@@
 	)
 	(segment
-		(start 125.501 55.905)
-		(end 127.405 55.905)
+		(start 85.09 55.88)
+		(end 75.692 55.88)
 		(width 1.6)
 		(layer "B.Cu")
@@
 	)
 	(segment
-		(start 124.968 56.388)
-		(end 125.476 55.88)
-		(width 1.6)
-		(layer "B.Cu")
-		(net "/WA")
-	)
-	(segment
 		(start 36.322 75.946)
 		(end 42.926 75.946)
@@
 	)
 	(segment
-		(start 126.517 58.445)
-		(end 127.405 58.445)
+		(start 104.634 58.42)
+		(end 111.389 58.42)
 		(width 1.6)
 		(layer "B.Cu")
@@
 	)
 	(segment
-		(start 104.634 58.42)
-		(end 111.389 58.42)
+		(start 70.358 59.944)
+		(end 54.61 59.944)
 		(width 1.6)
 		(layer "B.Cu")
@@
 	)
 	(segment
-		(start 70.358 59.944)
-		(end 54.61 59.944)
+		(start 115.316 58.42)
+		(end 115.57 58.674)
 		(width 1.6)
 		(layer "B.Cu")
@@
 	)
 	(segment
-		(start 126.492 58.42)
-		(end 126.517 58.445)
+		(start 40.894 73.66)
+		(end 38.1 73.66)
 		(width 1.6)
 		(layer "B.Cu")
@@
 	)
 	(segment
-		(start 40.894 73.66)
-		(end 38.1 73.66)
+		(start 115.57 58.674)
+		(end 126.492 58.674)
 		(width 1.6)
 		(layer "B.Cu")
@@
 	)
 	(segment
-		(start 115.316 58.42)
-		(end 115.57 58.674)
+		(start 127.405 58.445)
+		(end 126.721 58.445)
 		(width 1.6)
 		(layer "B.Cu")
@@
 	)
 	(segment
-		(start 114.3 58.42)
-		(end 115.316 58.42)
+		(start 126.721 58.445)
+		(end 126.492 58.674)
 		(width 1.6)
 		(layer "B.Cu")
@@
 	)
 	(segment
-		(start 115.57 58.674)
-		(end 126.238 58.674)
-		(width 1.6)
-		(layer "B.Cu")
-		(net "/WB")
-	)
-	(segment
-		(start 126.238 58.674)
-		(end 126.492 58.42)
+		(start 114.3 58.42)
+		(end 115.316 58.42)
 		(width 1.6)
 		(layer "B.Cu")
